Commit message: Update arduino_robot_arm.urdf

File: urdf.afterEdit/arduino_robot_arm.urdf (robot description, URDF)
Before this commit: robot arduino_robot_arm, 5 links, 4 joints
Joints:
- joint elbow: limit lower=-1.57 upper=1.57 effort=1000.0 velocity=1.0 -> lower=-2.5 upper=2.5 effort=1000.0 velocity=1.0
